Commit message: v1: 9+1 DOF arm verified

File: urdf/myrobot.urdf.xacro (robot description, xacro)
@@ -1,6 +1,6 @@
 <?xml version="1.0"?>
-<robot name="myrobot_10dof" xmlns:xacro="http://ros.org/wiki/xacro">
-  <xacro:include filename="$(find myrobot_10dof_description)/urdf/myrobot_10dof.xacro"/>
-  <xacro:include filename="$(find myrobot_10dof_description)/urdf/myrobot_10dof_hand.xacro"/>
+<robot name="myrobot" xmlns:xacro="http://ros.org/wiki/xacro">
+  <xacro:include filename="$(find myrobot_description)/urdf/myrobot.xacro"/>
+  <xacro:include filename="$(find myrobot_description)/urdf/myrobot_hand.xacro"/>
   <!-- setting color -->
   <material name="white">
@@ -21,5 +21,5 @@
   </xacro:if>
   <xacro:if value="$(arg use_gazebo_simulation)">
-    <xacro:include filename="$(find myrobot_10dof_description)/urdf/myrobot_10dof_gazebo.xacro"/>
+    <xacro:include filename="$(find myrobot_description)/urdf/myrobot_gazebo.xacro"/>
     <xacro:if value="$(arg load_trans1)">
       <!-- <xacro:default_transmission joint_name="arm_joint01" interface="${right_arm_interface}"/> -->
@@ -45,5 +45,5 @@
     <origin xyz="0 0 1.5" rpy="0 0 0"/>
   </joint>
-  <xacro:myrobot_10dof
+  <xacro:myrobot
     arm_joint1_lower_limit="${radians(-90)}"
     arm_joint1_upper_limit="${radians(90)}"
@@ -69,6 +69,6 @@
     arm_joints_velocity_limit="${VELOCITY_LIMIT}"
     arm_color="white">
-  </xacro:myrobot_10dof>
-  <xacro:myrobot_10dof_hand
+  </xacro:myrobot>
+  <xacro:myrobot_hand
     hand_joints_lower_limit="${radians(-90)}"
     hand_joints_upper_limit="${radians(0)}"
@@ -76,4 +76,4 @@
     hand_joints_velocity_limit="${VELOCITY_LIMIT}"
     hand_color="red">
-  </xacro:myrobot_10dof_hand>
+  </xacro:myrobot_hand>
 </robot>

File: urdf/myrobot.xacro (robot description, xacro)
@@ -1,5 +1,5 @@
 <?xml version="1.0"?>
 <robot xmlns:xacro="http://ros.org/wiki/xacro">
-  <xacro:macro name="myrobot_10dof"
+  <xacro:macro name="myrobot"
     params="arm_joint1_lower_limit
             arm_joint1_upper_limit
@@ -36,12 +36,12 @@
         <origin rpy="3.14159 0 0" xyz="0 0 0"/>
         <geometry>
-          <mesh filename="package://myrobot_10dof_description/meshes/visual/com1.stl" scale="0.001 0.001 0.001"/>
-        </geometry>
-        <material name="${arm_color}"/>
-      </visual>
-      <collision>
-        <origin rpy="3.14159 0 0" xyz="0 0 0"/>
-        <geometry>
-          <mesh filename="package://myrobot_10dof_description/meshes/collision/com1.stl" scale="0.001 0.001 0.001"/>
+          <mesh filename="package://myrobot_description/meshes/visual/com1.stl" scale="0.001 0.001 0.001"/>
+        </geometry>
+        <material name="${arm_color}"/>
+      </visual>
+      <collision>
+        <origin rpy="3.14159 0 0" xyz="0 0 0"/>
+        <geometry>
+          <mesh filename="package://myrobot_description/meshes/collision/com1.stl" scale="0.001 0.001 0.001"/>
         </geometry>
       </collision>
@@ -65,12 +65,12 @@
         <origin rpy="3.14159 0 0" xyz="0 0 0"/>
         <geometry>
-          <mesh filename="package://myrobot_10dof_description/meshes/visual/com2.stl" scale="0.001 0.001 0.001"/>
-        </geometry>
-        <material name="${arm_color}"/>
-      </visual>
-      <collision>
-        <origin rpy="3.14159 0 0" xyz="0 0 0"/>
-        <geometry>
-          <mesh filename="package://myrobot_10dof_description/meshes/collision/com2.stl" scale="0.001 0.001 0.001"/>
+          <mesh filename="package://myrobot_description/meshes/visual/com2.stl" scale="0.001 0.001 0.001"/>
+        </geometry>
+        <material name="${arm_color}"/>
+      </visual>
+      <collision>
+        <origin rpy="3.14159 0 0" xyz="0 0 0"/>
+        <geometry>
+          <mesh filename="package://myrobot_description/meshes/collision/com2.stl" scale="0.001 0.001 0.001"/>
         </geometry>
       </collision>
@@ -94,12 +94,12 @@
         <origin rpy="3.14159 0 0" xyz="0 0 0"/>
         <geometry>
-          <mesh filename="package://myrobot_10dof_description/meshes/visual/com3.stl" scale="0.001 0.001 0.001"/>
-        </geometry>
-        <material name="${arm_color}"/>
-      </visual>
-      <collision>
-        <origin rpy="3.14159 0 0" xyz="0 0 0"/>
-        <geometry>
-          <mesh filename="package://myrobot_10dof_description/meshes/collision/com3.stl" scale="0.001 0.001 0.001"/>
+          <mesh filename="package://myrobot_description/meshes/visual/com3.stl" scale="0.001 0.001 0.001"/>
+        </geometry>
+        <material name="${arm_color}"/>
+      </visual>
+      <collision>
+        <origin rpy="3.14159 0 0" xyz="0 0 0"/>
+        <geometry>
+          <mesh filename="package://myrobot_description/meshes/collision/com3.stl" scale="0.001 0.001 0.001"/>
         </geometry>
       </collision>
@@ -123,12 +123,12 @@
         <origin rpy="3.14159 0 0" xyz="0 0 0"/>
         <geometry>
-          <mesh filename="package://myrobot_10dof_description/meshes/visual/com4.stl" scale="0.001 0.001 0.001"/>
-        </geometry>
-        <material name="${arm_color}"/>
-      </visual>
-      <collision>
-        <origin rpy="3.14159 0 0" xyz="0 0 0"/>
-        <geometry>
-          <mesh filename="package://myrobot_10dof_description/meshes/collision/com4.stl" scale="0.001 0.001 0.001"/>
+          <mesh filename="package://myrobot_description/meshes/visual/com4.stl" scale="0.001 0.001 0.001"/>
+        </geometry>
+        <material name="${arm_color}"/>
+      </visual>
+      <collision>
+        <origin rpy="3.14159 0 0" xyz="0 0 0"/>
+        <geometry>
+          <mesh filename="package://myrobot_description/meshes/collision/com4.stl" scale="0.001 0.001 0.001"/>
         </geometry>
       </collision>
@@ -152,12 +152,12 @@
         <origin rpy="3.14159 0 0" xyz="0 0 0"/>
         <geometry>
-          <mesh filename="package://myrobot_10dof_description/meshes/visual/com5.stl" scale="0.001 0.001 0.001"/>
-        </geometry>
-        <material name="${arm_color}"/>
-      </visual>
-      <collision>
-        <origin rpy="3.14159 0 0" xyz="0 0 0"/>
-        <geometry>
-          <mesh filename="package://myrobot_10dof_description/meshes/collision/com5.stl" scale="0.001 0.001 0.001"/>
+          <mesh filename="package://myrobot_description/meshes/visual/com5.stl" scale="0.001 0.001 0.001"/>
+        </geometry>
+        <material name="${arm_color}"/>
+      </visual>
+      <collision>
+        <origin rpy="3.14159 0 0" xyz="0 0 0"/>
+        <geometry>
+          <mesh filename="package://myrobot_description/meshes/collision/com5.stl" scale="0.001 0.001 0.001"/>
         </geometry>
       </collision>
@@ -181,12 +181,12 @@
         <origin rpy="3.14159 0 0" xyz="0 0 0"/>
         <geometry>
-          <mesh filename="package://myrobot_10dof_description/meshes/visual/com6.stl" scale="0.001 0.001 0.001"/>
-        </geometry>
-        <material name="${arm_color}"/>
-      </visual>
-      <collision>
-        <origin rpy="3.14159 0 0" xyz="0 0 0"/>
-        <geometry>
-          <mesh filename="package://myrobot_10dof_description/meshes/collision/com6.stl" scale="0.001 0.001 0.001"/>
+          <mesh filename="package://myrobot_description/meshes/visual/com6.stl" scale="0.001 0.001 0.001"/>
+        </geometry>
+        <material name="${arm_color}"/>
+      </visual>
+      <collision>
+        <origin rpy="3.14159 0 0" xyz="0 0 0"/>
+        <geometry>
+          <mesh filename="package://myrobot_description/meshes/collision/com6.stl" scale="0.001 0.001 0.001"/>
         </geometry>
       </collision>
@@ -210,12 +210,12 @@
         <origin rpy="3.14159 0 0" xyz="0 0 0"/>
         <geometry>
-          <mesh filename="package://myrobot_10dof_description/meshes/visual/com7.stl" scale="0.001 0.001 0.001"/>
-        </geometry>
-        <material name="${arm_color}"/>
-      </visual>
-      <collision>
-        <origin rpy="3.14159 0 0" xyz="0 0 0"/>
-        <geometry>
-          <mesh filename="package://myrobot_10dof_description/meshes/collision/com7.stl" scale="0.001 0.001 0.001"/>
+          <mesh filename="package://myrobot_description/meshes/visual/com7.stl" scale="0.001 0.001 0.001"/>
+        </geometry>
+        <material name="${arm_color}"/>
+      </visual>
+      <collision>
+        <origin rpy="3.14159 0 0" xyz="0 0 0"/>
+        <geometry>
+          <mesh filename="package://myrobot_description/meshes/collision/com7.stl" scale="0.001 0.001 0.001"/>
         </geometry>
       </collision>
@@ -239,12 +239,12 @@
         <origin rpy="3.14159 0 0" xyz="0 0 0"/>
         <geometry>
-          <mesh filename="package://myrobot_10dof_description/meshes/visual/com8.stl" scale="0.001 0.001 0.001"/>
-        </geometry>
-        <material name="${arm_color}"/>
-      </visual>
-      <collision>
-        <origin rpy="3.14159 0 0" xyz="0 0 0"/>
-        <geometry>
-          <mesh filename="package://myrobot_10dof_description/meshes/collision/com8.stl" scale="0.001 0.001 0.001"/>
+          <mesh filename="package://myrobot_description/meshes/visual/com8.stl" scale="0.001 0.001 0.001"/>
+        </geometry>
+        <material name="${arm_color}"/>
+      </visual>
+      <collision>
+        <origin rpy="3.14159 0 0" xyz="0 0 0"/>
+        <geometry>
+          <mesh filename="package://myrobot_description/meshes/collision/com8.stl" scale="0.001 0.001 0.001"/>
         </geometry>
       </collision>
@@ -268,12 +268,12 @@
         <origin rpy="3.14159 0 0" xyz="0 0 0"/>
         <geometry>
-          <mesh filename="package://myrobot_10dof_description/meshes/visual/com9.stl" scale="0.001 0.001 0.001"/>
-        </geometry>
-        <material name="${arm_color}"/>
-      </visual>
-      <collision>
-        <origin rpy="3.14159 0 0" xyz="0 0 0"/>
-        <geometry>
-          <mesh filename="package://myrobot_10dof_description/meshes/collision/com9.stl" scale="0.001 0.001 0.001"/>
+          <mesh filename="package://myrobot_description/meshes/visual/com9.stl" scale="0.001 0.001 0.001"/>
+        </geometry>
+        <material name="${arm_color}"/>
+      </visual>
+      <collision>
+        <origin rpy="3.14159 0 0" xyz="0 0 0"/>
+        <geometry>
+          <mesh filename="package://myrobot_description/meshes/collision/com9.stl" scale="0.001 0.001 0.001"/>
         </geometry>
       </collision>

File: urdf/myrobot_hand.xacro (robot description, xacro)
@@ -1,5 +1,5 @@
 <?xml version="1.0"?>
 <robot xmlns:xacro="http://ros.org/wiki/xacro">
-  <xacro:macro name="myrobot_10dof_hand"
+  <xacro:macro name="myrobot_hand"
     params="hand_joints_lower_limit
             hand_joints_upper_limit
@@ -12,5 +12,5 @@
         <origin rpy="3.14159 0 1.5708" xyz="0.0 0.0 0.0"/>
         <geometry>
-          <mesh filename="package://myrobot_10dof_description/meshes/visual/com10C.stl" scale="0.001 0.001 0.001"/>
+          <mesh filename="package://myrobot_description/meshes/visual/com10C.stl" scale="0.001 0.001 0.001"/>
         </geometry>
         <material name="${hand_color}"/>
@@ -19,5 +19,5 @@
         <origin rpy="3.14159 0 1.5708" xyz="0.0 0.0 0.0"/>
         <geometry>
-          <mesh filename="package://myrobot_10dof_description/meshes/collision/com10C.stl" scale="0.001 0.001 0.001"/>
+          <mesh filename="package://myrobot_description/meshes/collision/com10C.stl" scale="0.001 0.001 0.001"/>
         </geometry>
       </collision>
@@ -44,5 +44,5 @@
         <origin rpy="3.14159 0 -1.5708" xyz="0.0 0.0 0.0"/>
         <geometry>
-          <mesh filename="package://myrobot_10dof_description/meshes/visual/com10A.stl" scale="0.001 0.001 0.001"/>
+          <mesh filename="package://myrobot_description/meshes/visual/com10A.stl" scale="0.001 0.001 0.001"/>
         </geometry>
         <material name="${hand_color}"/>
@@ -51,5 +51,5 @@
         <origin rpy="3.14159 0 -1.5708" xyz="0.0 0.0 0.0"/>
         <geometry>
-          <mesh filename="package://myrobot_10dof_description/meshes/collision/com10A.stl" scale="0.001 0.001 0.001"/>
+          <mesh filename="package://myrobot_description/meshes/collision/com10A.stl" scale="0.001 0.001 0.001"/>
         </geometry>
       </collision>
@@ -77,5 +77,5 @@
         <origin rpy="3.14159 0 -1.5708" xyz="0.0 0.0 0.0"/>
         <geometry>
-          <mesh filename="package://myrobot_10dof_description/meshes/visual/com10B.stl" scale="0.001 0.001 0.001"/>
+          <mesh filename="package://myrobot_description/meshes/visual/com10B.stl" scale="0.001 0.001 0.001"/>
         </geometry>
         <material name="${hand_color}"/>
@@ -84,5 +84,5 @@
         <origin rpy="3.14159 0 -1.5708" xyz="0.0 0.0 0.0"/>
         <geometry>
-          <mesh filename="package://myrobot_10dof_description/meshes/collision/com10B.stl" scale="0.001 0.001 0.001"/>
+          <mesh filename="package://myrobot_description/meshes/collision/com10B.stl" scale="0.001 0.001 0.001"/>
         </geometry>
       </collision>

File: urdf/sciurus17_right_arm_only.urdf.xacro (robot description, xacro)
@@ -1,6 +1,6 @@
 <?xml version="1.0"?>
 <robot name="sciurus17" xmlns:xacro="http://ros.org/wiki/xacro">
-  <xacro:include filename="$(find myrobot_10dof_description)/urdf/sciurus17_right_arm_only.xacro"/>
-  <xacro:include filename="$(find myrobot_10dof_description)/urdf/sciurus17_right_hand.xacro"/>
+  <xacro:include filename="$(find myrobot_description)/urdf/sciurus17_right_arm_only.xacro"/>
+  <xacro:include filename="$(find myrobot_description)/urdf/sciurus17_right_hand.xacro"/>
   <!-- setting color -->
   <material name="white">
@@ -21,5 +21,5 @@
   </xacro:if>
   <xacro:if value="$(arg use_gazebo_simulation)">
-    <xacro:include filename="$(find myrobot_10dof_description)/urdf/sciurus17_gazebo.xacro"/>
+    <xacro:include filename="$(find myrobot_description)/urdf/sciurus17_gazebo.xacro"/>
     <xacro:if value="$(arg load_trans1)">
       <xacro:default_transmission joint_name="r_arm_joint1" interface="${right_arm_interface}"/>

File: urdf/sciurus17_right_arm_only.xacro (robot description, xacro)
@@ -36,12 +36,12 @@
         <origin rpy="1.5708 0 0" xyz="0.0 0.0 0.0"/>
         <geometry>
-          <mesh filename="package://myrobot_10dof_description/meshes/visual/R_Link1.stl" scale="1.0 1.0 1.0"/>
-        </geometry>
-        <material name="${arm_color}"/>
-      </visual>
-      <collision>
-        <origin rpy="1.5708 0 0" xyz="0.0 0.0 0.0"/>
-        <geometry>
-          <mesh filename="package://myrobot_10dof_description/meshes/collision/R_Link1.stl" scale="1.0 1.0 1.0"/>
+          <mesh filename="package://myrobot_description/meshes/visual/R_Link1.stl" scale="1.0 1.0 1.0"/>
+        </geometry>
+        <material name="${arm_color}"/>
+      </visual>
+      <collision>
+        <origin rpy="1.5708 0 0" xyz="0.0 0.0 0.0"/>
+        <geometry>
+          <mesh filename="package://myrobot_description/meshes/collision/R_Link1.stl" scale="1.0 1.0 1.0"/>
         </geometry>
       </collision>
@@ -68,5 +68,5 @@
         <origin rpy="0 1.5708 0" xyz="0.0 0.0 0.0"/>
         <geometry>
-          <mesh filename="package://myrobot_10dof_description/meshes/visual/R_Link2.stl" scale="1.0 1.0 1.0"/>
+          <mesh filename="package://myrobot_description/meshes/visual/R_Link2.stl" scale="1.0 1.0 1.0"/>
         </geometry>
         <material name="${arm_color}"/>
@@ -75,5 +75,5 @@
         <origin rpy="0 1.5708 0" xyz="0.0 0.0 0.0"/>
         <geometry>
-          <mesh filename="package://myrobot_10dof_description/meshes/collision/R_Link2.stl" scale="1.0 1.0 1.0"/>
+          <mesh filename="package://myrobot_description/meshes/collision/R_Link2.stl" scale="1.0 1.0 1.0"/>
         </geometry>
       </collision>
@@ -100,12 +100,12 @@
         <origin rpy="1.5708 0 0" xyz="0.0 0.0 0.0"/>
         <geometry>
-          <mesh filename="package://myrobot_10dof_description/meshes/visual/L_Link3.stl" scale="1.0 -1.0 1.0"/>
-        </geometry>
-        <material name="${arm_color}"/>
-      </visual>
-      <collision>
-        <origin rpy="1.5708 0 0" xyz="0.0 0.0 0.0"/>
-        <geometry>
-          <mesh filename="package://myrobot_10dof_description/meshes/collision/L_Link3.stl" scale="1.0 -1.0 1.0"/>
+          <mesh filename="package://myrobot_description/meshes/visual/L_Link3.stl" scale="1.0 -1.0 1.0"/>
+        </geometry>
+        <material name="${arm_color}"/>
+      </visual>
+      <collision>
+        <origin rpy="1.5708 0 0" xyz="0.0 0.0 0.0"/>
+        <geometry>
+          <mesh filename="package://myrobot_description/meshes/collision/L_Link3.stl" scale="1.0 -1.0 1.0"/>
         </geometry>
       </collision>
@@ -132,12 +132,12 @@
         <origin rpy="0 0 0" xyz="0.0 0.0 0.0"/>
         <geometry>
-          <mesh filename="package://myrobot_10dof_description/meshes/visual/R_Link4.stl" scale="1.0 1.0 1.0"/>
-        </geometry>
-        <material name="${arm_color}"/>
-      </visual>
-      <collision>
-        <origin rpy="0 0 0" xyz="0.0 0.0 0.0"/>
-        <geometry>
-          <mesh filename="package://myrobot_10dof_description/meshes/collision/R_Link4.stl" scale="1.0 1.0 1.0"/>
+          <mesh filename="package://myrobot_description/meshes/visual/R_Link4.stl" scale="1.0 1.0 1.0"/>
+        </geometry>
+        <material name="${arm_color}"/>
+      </visual>
+      <collision>
+        <origin rpy="0 0 0" xyz="0.0 0.0 0.0"/>
+        <geometry>
+          <mesh filename="package://myrobot_description/meshes/collision/R_Link4.stl" scale="1.0 1.0 1.0"/>
         </geometry>
       </collision>
@@ -164,5 +164,5 @@
         <origin rpy="1.5708 0 0" xyz="0.0 0.0 0.0"/>
         <geometry>
-          <mesh filename="package://myrobot_10dof_description/meshes/visual/R_Link5.stl" scale="1.0 1.0 1.0"/>
+          <mesh filename="package://myrobot_description/meshes/visual/R_Link5.stl" scale="1.0 1.0 1.0"/>
         </geometry>
         <material name="${arm_color}"/>
@@ -171,5 +171,5 @@
         <origin xyz="0.032 -0.074 0.0345" rpy="0 0 -2.0944"/>
         <geometry>
-          <mesh filename="package://myrobot_10dof_description/meshes/visual/Logo_Rabbit.stl" scale="1.0 1.0 1.0"/>
+          <mesh filename="package://myrobot_description/meshes/visual/Logo_Rabbit.stl" scale="1.0 1.0 1.0"/>
         </geometry>
         <material name="red_color">
@@ -180,5 +180,5 @@
         <origin xyz="0.013 -0.107 0.0345" rpy="0 0 -2.0944"/>
         <geometry>
-          <mesh filename="package://myrobot_10dof_description/meshes/visual/Logo_Corp.stl" scale="1.0 1.0 1.0"/>
+          <mesh filename="package://myrobot_description/meshes/visual/Logo_Corp.stl" scale="1.0 1.0 1.0"/>
         </geometry>
         <material name="black_color">
@@ -189,5 +189,5 @@
         <origin rpy="1.5708 0 0" xyz="0.0 0.0 0.0"/>
         <geometry>
-          <mesh filename="package://myrobot_10dof_description/meshes/collision/R_Link5.stl" scale="1.0 1.0 1.0"/>
+          <mesh filename="package://myrobot_description/meshes/collision/R_Link5.stl" scale="1.0 1.0 1.0"/>
         </geometry>
       </collision>
@@ -234,12 +234,12 @@
         <origin rpy="0 0 0" xyz="0.0 0.0 0.0"/>
         <geometry>
-          <mesh filename="package://myrobot_10dof_description/meshes/visual/R_Link6.stl" scale="1.0 1.0 1.0"/>
-        </geometry>
-        <material name="${arm_color}"/>
-      </visual>
-      <collision>
-        <origin rpy="0 0 0" xyz="0.0 0.0 0.0"/>
-        <geometry>
-          <mesh filename="package://myrobot_10dof_description/meshes/collision/R_Link6.stl" scale="1.0 1.0 1.0"/>
+          <mesh filename="package://myrobot_description/meshes/visual/R_Link6.stl" scale="1.0 1.0 1.0"/>
+        </geometry>
+        <material name="${arm_color}"/>
+      </visual>
+      <collision>
+        <origin rpy="0 0 0" xyz="0.0 0.0 0.0"/>
+        <geometry>
+          <mesh filename="package://myrobot_description/meshes/collision/R_Link6.stl" scale="1.0 1.0 1.0"/>
         </geometry>
       </collision>
