Commit message: v2: arm failed to move due to excessive weight

File: urdf/myrobot.xacro (robot description, xacro)
@@ -2,39 +2,47 @@
 <robot xmlns:xacro="http://ros.org/wiki/xacro">
   <xacro:macro name="myrobot"
-    params="arm_joint1_lower_limit
-            arm_joint1_upper_limit
-            arm_joint2_lower_limit
-            arm_joint2_upper_limit
-            arm_joint3_lower_limit
-            arm_joint3_upper_limit
-            arm_joint4_lower_limit
-            arm_joint4_upper_limit
-            arm_joint5_lower_limit
-            arm_joint5_upper_limit
-            arm_joint6_lower_limit
-            arm_joint6_upper_limit
-            arm_joint7_lower_limit
-            arm_joint7_upper_limit
-            arm_joint8_lower_limit
-            arm_joint8_upper_limit
-            arm_joint9_lower_limit
-            arm_joint9_upper_limit
-            arm_joint10_lower_limit
-            arm_joint10_upper_limit
-            arm_joints_effort_limit
-            arm_joints_velocity_limit
+    params="joint01_lower_limit
+            joint01_upper_limit
+            joint02_lower_limit
+            joint02_upper_limit
+            joint03_lower_limit
+            joint03_upper_limit
+            joint04_lower_limit
+            joint04_upper_limit
+            joint05_lower_limit
+            joint05_upper_limit
+            joint06_lower_limit
+            joint06_upper_limit
+            joint07_lower_limit
+            joint07_upper_limit
+            joint08_lower_limit
+            joint08_upper_limit
+            joint09_lower_limit
+            joint09_upper_limit
+            joint10_lower_limit
+            joint10_upper_limit
+            joint01_effort_limit joint01_velocity_limit
+            joint02_effort_limit joint02_velocity_limit
+            joint03_effort_limit joint03_velocity_limit
+            joint04_effort_limit joint04_velocity_limit
+            joint05_effort_limit joint05_velocity_limit
+            joint06_effort_limit joint06_velocity_limit
+            joint07_effort_limit joint07_velocity_limit
+            joint08_effort_limit joint08_velocity_limit
+            joint09_effort_limit joint09_velocity_limit
+            joint10_effort_limit joint10_velocity_limit
             arm_color
             ">
-    <!-- ================= Link 1 ================= -->
-    <joint name="arm_joint01" type="fixed">
+    <!-- ================= Joint 0 ================= -->
+    <joint name="arm_base_fixed_joint" type="fixed">
       <parent link="base_link" />
-      <child link="link1" />
+      <child link="link01" />
       <origin xyz="0 0 0" rpy="0 0 0"/>
     </joint>
-    <link name="link1">
+    <link name="link01">
       <visual>
         <origin rpy="3.14159 0 0" xyz="0 0 0"/>
         <geometry>
-          <mesh filename="package://myrobot_description/meshes/visual/com1.stl" scale="0.001 0.001 0.001"/>
+          <mesh filename="package://myrobot_description/meshes/visual/com01.stl" scale="0.001 0.001 0.001"/>
         </geometry>
         <material name="${arm_color}"/>
@@ -43,27 +51,27 @@
         <origin rpy="3.14159 0 0" xyz="0 0 0"/>
         <geometry>
-          <mesh filename="package://myrobot_description/meshes/collision/com1.stl" scale="0.001 0.001 0.001"/>
-        </geometry>
-      </collision>
-      <inertial>
-        <origin rpy="0 0 0" xyz="0 0 0"/>
-        <inertia ixx="1e-4" ixy="0" ixz="0" iyy="1e-4" iyz="0" izz="1e-4"/>
-        <mass value="0.25"/>
-      </inertial>
-    </link>
-    <!-- ================= Link 2 ================= -->
-    <joint name="arm_joint02" type="revolute">
-      <parent link="link1" />
-      <child link="link2" />
-      <origin xyz="0 0 -0.0715" rpy="0 0 0"/>
-      <limit lower="${arm_joint2_lower_limit}" upper="${arm_joint2_upper_limit}" effort="${arm_joints_effort_limit}" velocity="${arm_joints_velocity_limit}"/>
+          <mesh filename="package://myrobot_description/meshes/collision/com01.stl" scale="0.001 0.001 0.001"/>
+        </geometry>
+      </collision>
+      <inertial>
+        <origin xyz="2.529e-12 0 0.040805" rpy="0 0 0"/>
+        <mass value="0.987927"/>
+        <inertia ixx="0.001363" ixy="1.036e-18" ixz="-2.991e-15" iyy="0.001363" iyz="0" izz="0.001426"/>
+      </inertial>
+    </link>
+    <!-- ================= Joint 1 ================= -->
+    <joint name="joint01" type="revolute">
+      <parent link="link01" />
+      <child link="link02" />00
+      <origin xyz="0 0 -0.084" rpy="0 0 0"/>
+      <limit lower="${joint01_lower_limit}" upper="${joint01_upper_limit}" effort="${joint01_effort_limit}" velocity="${joint01_velocity_limit}"/>
       <axis xyz="0 0 1"/>
       <dynamics damping="1.0e-6" friction="0.8"/>
     </joint>
-    <link name="link2">
+    <link name="link02">
       <visual>
         <origin rpy="3.14159 0 0" xyz="0 0 0"/>
         <geometry>
-          <mesh filename="package://myrobot_description/meshes/visual/com2.stl" scale="0.001 0.001 0.001"/>
+          <mesh filename="package://myrobot_description/meshes/visual/com02.stl" scale="0.001 0.001 0.001"/>
         </geometry>
         <material name="${arm_color}"/>
@@ -72,222 +80,260 @@
         <origin rpy="3.14159 0 0" xyz="0 0 0"/>
         <geometry>
-          <mesh filename="package://myrobot_description/meshes/collision/com2.stl" scale="0.001 0.001 0.001"/>
-        </geometry>
-      </collision>
-      <inertial>
-        <origin rpy="0 0 0" xyz="0 0 0"/>
-        <inertia ixx="1e-4" ixy="0" ixz="0" iyy="1e-4" iyz="0" izz="1e-4"/>
-        <mass value="0.2"/>
-      </inertial>
-    </link>
-    <!-- ================= Link 3 ================= -->
-    <joint name="arm_joint03" type="revolute">
-      <parent link="link2" />
-      <child link="link3" />
-      <origin xyz="0 0 -0.08" rpy="0 0 0"/>
-      <limit lower="${arm_joint3_lower_limit}" upper="${arm_joint3_upper_limit}" effort="${arm_joints_effort_limit}" velocity="${arm_joints_velocity_limit}"/>
-      <axis xyz="0 1 0"/>
-      <dynamics damping="1.0e-6" friction="0.8"/>
-    </joint>
-    <link name="link3">
-      <visual>
-        <origin rpy="3.14159 0 0" xyz="0 0 0"/>
-        <geometry>
-          <mesh filename="package://myrobot_description/meshes/visual/com3.stl" scale="0.001 0.001 0.001"/>
-        </geometry>
-        <material name="${arm_color}"/>
-      </visual>
-      <collision>
-        <origin rpy="3.14159 0 0" xyz="0 0 0"/>
-        <geometry>
-          <mesh filename="package://myrobot_description/meshes/collision/com3.stl" scale="0.001 0.001 0.001"/>
-        </geometry>
-      </collision>
-      <inertial>
-        <origin rpy="0 0 0" xyz="0 0 0"/>
-        <inertia ixx="1e-4" ixy="0" ixz="0" iyy="1e-4" iyz="0" izz="1e-4"/>
-        <mass value="0.2"/>
-      </inertial>
-    </link>
-    <!-- ================= Link 4 ================= -->
-    <joint name="arm_joint04" type="revolute">
-      <parent link="link3" />
-      <child link="link4" />
-      <origin xyz="0 0 -0.2265" rpy="0 0 0"/>
-      <limit lower="${arm_joint4_lower_limit}" upper="${arm_joint4_upper_limit}" effort="${arm_joints_effort_limit}" velocity="${arm_joints_velocity_limit}"/>
+          <mesh filename="package://myrobot_description/meshes/collision/com02.stl" scale="0.001 0.001 0.001"/>
+        </geometry>
+      </collision>
+      <inertial>
+        <origin xyz="0.001015 1.837e-12 0.031665" rpy="0 0 0"/>
+        <mass value="0.705618"/>
+        <inertia ixx="0.0004845" ixy="-4.897e-15" ixz="-4.179279e-6"
+                iyy="0.0005896" iyz="-7.564e-15" izz="0.0006012"/>
+      </inertial>
+    </link>
+    <!-- ================= Joint 2  ================= -->
+    <joint name="joint02" type="revolute">
+      <parent link="link02"/>
+      <child link="link03"/>
+      <origin xyz="0 0 -0.0385" rpy="0 0 0"/>
+      <limit lower="${joint02_lower_limit}" upper="${joint02_upper_limit}" effort="${joint02_effort_limit}" velocity="${joint02_velocity_limit}"/>
+      <axis xyz="1 0 0"/>
+      <dynamics damping="1.0e-6" friction="0.8"/>
+    </joint>
+    <link name="link03">
+      <visual>
+        <origin rpy="3.14159 0 0" xyz="0 0 -0.370"/>
+        <geometry>
+          <mesh filename="package://myrobot_description/meshes/visual/com03.stl" scale="0.001 0.001 0.001"/>
+        </geometry>
+        <material name="${arm_color}"/>
+      </visual>
+      <collision>
+        <origin rpy="3.14159 0 0" xyz="0 0 -0.370"/>
+        <geometry>
+          <mesh filename="package://myrobot_description/meshes/collision/com03.stl" scale="0.001 0.001 0.001"/>
+        </geometry>
+      </collision>
+      <inertial>
+        <origin xyz="-0.00029 -2.571e-13 -0.135978" rpy="0 0 0"/>
+        <mass value="2.518019"/>
+        <inertia ixx="0.03772" ixy="-1.633e-15" ixz="9.9423617e-5"
+                iyy="0.04126" iyz="8.79e-14" izz="0.00532"/>
+      </inertial>
+    </link>
+    <!-- ================= Joint 3 ================= -->
+    <joint name="joint03" type="revolute">
+      <parent link="link03" />
+      <child link="link04" />
+      <origin xyz="0 0 -0.370" rpy="0 0 0"/>
+      <limit lower="${joint03_lower_limit}" upper="${joint03_upper_limit}" effort="${joint03_effort_limit}" velocity="${joint03_velocity_limit}"/>
+      <axis xyz="1 0 0"/>
+      <dynamics damping="1.0e-6" friction="0.8"/>
+    </joint>
+    <link name="link04">
+      <visual>
+        <origin rpy="3.14159 0 0" xyz="0 0 -0.300"/>
+        <geometry>
+          <mesh filename="package://myrobot_description/meshes/visual/com04.stl" scale="0.001 0.001 0.001"/>
+        </geometry>
+        <material name="${arm_color}"/>
+      </visual>
+      <collision>
+        <origin rpy="3.14159 0 0" xyz="0 0 -0.300"/>
+        <geometry>
+          <mesh filename="package://myrobot_description/meshes/collision/com04.stl" scale="0.001 0.001 0.001"/>
+        </geometry>
+      </collision>
+      <inertial>
+        <origin xyz="-0.000228 0.001307 -0.053587" rpy="0 0 0"/>
+        <mass value="2.663893"/>
+        <inertia ixx="0.04266" ixy="-7.95006e-7" ixz="-3.3404576e-5"
+                iyy="0.04593" iyz="-0.0004672" izz="0.006191"/>
+      </inertial>
+    </link>
+    <!-- ================= Joint 4 ================= -->
+    <joint name="joint04" type="revolute">
+      <parent link="link04" />
+      <child link="link05" />
+      <origin xyz="0 0 -0.4099" rpy="0 0 0"/>
+      <limit lower="${joint04_lower_limit}" upper="${joint04_upper_limit}" effort="${joint04_effort_limit}" velocity="${joint04_velocity_limit}"/>
       <axis xyz="0 0 1"/>
       <dynamics damping="1.0e-6" friction="0.8"/>
     </joint>
-    <link name="link4">
-      <visual>
-        <origin rpy="3.14159 0 0" xyz="0 0 0"/>
-        <geometry>
-          <mesh filename="package://myrobot_description/meshes/visual/com4.stl" scale="0.001 0.001 0.001"/>
-        </geometry>
-        <material name="${arm_color}"/>
-      </visual>
-      <collision>
-        <origin rpy="3.14159 0 0" xyz="0 0 0"/>
-        <geometry>
-          <mesh filename="package://myrobot_description/meshes/collision/com4.stl" scale="0.001 0.001 0.001"/>
-        </geometry>
-      </collision>
-      <inertial>
-        <origin rpy="0 0 0" xyz="0 0 0"/>
-        <inertia ixx="1e-4" ixy="0" ixz="0" iyy="1e-4" iyz="0" izz="1e-4"/>
-        <mass value="0.2"/>
-      </inertial>
-    </link>
-    <!-- ================= Link 5 ================= -->
-    <joint name="arm_joint05" type="revolute">
-      <parent link="link4" />
-      <child link="link5" />
-      <origin xyz="0 0 -0.150" rpy="0 0 0"/>
-      <limit lower="${arm_joint5_lower_limit}" upper="${arm_joint5_upper_limit}" effort="${arm_joints_effort_limit}" velocity="${arm_joints_velocity_limit}"/>
-      <axis xyz="0 1 0"/>
-      <dynamics damping="1.0e-6" friction="0.8"/>
-    </joint>
-    <link name="link5">
-      <visual>
-        <origin rpy="3.14159 0 0" xyz="0 0 0"/>
-        <geometry>
-          <mesh filename="package://myrobot_description/meshes/visual/com5.stl" scale="0.001 0.001 0.001"/>
-        </geometry>
-        <material name="${arm_color}"/>
-      </visual>
-      <collision>
-        <origin rpy="3.14159 0 0" xyz="0 0 0"/>
-        <geometry>
-          <mesh filename="package://myrobot_description/meshes/collision/com5.stl" scale="0.001 0.001 0.001"/>
-        </geometry>
-      </collision>
-      <inertial>
-        <origin rpy="0 0 0" xyz="0 0 0"/>
-        <inertia ixx="1e-4" ixy="0" ixz="0" iyy="1e-4" iyz="0" izz="1e-4"/>
-        <mass value="0.2"/>
-      </inertial>
-    </link>
-    <!-- ================= Link 6 ================= -->
-    <joint name="arm_joint06" type="revolute">
-      <parent link="link5" />
-      <child link="link6" />
-      <origin xyz="0 0 -0.2005" rpy="0 0 0"/>
-      <limit lower="${arm_joint6_lower_limit}" upper="${arm_joint6_upper_limit}" effort="${arm_joints_effort_limit}" velocity="${arm_joints_velocity_limit}"/>
+    <link name="link05">
+      <visual>
+        <origin rpy="3.14159 0 0" xyz="0 0 -0.005"/>
+        <geometry>
+          <mesh filename="package://myrobot_description/meshes/visual/com05.stl" scale="0.001 0.001 0.001"/>
+        </geometry>
+        <material name="${arm_color}"/>
+      </visual>
+      <collision>
+        <origin rpy="3.14159 0 0" xyz="0 0 -0.005"/>
+        <geometry>
+          <mesh filename="package://myrobot_description/meshes/collision/com05.stl" scale="0.001 0.001 0.001"/>
+        </geometry>
+      </collision>
+      <inertial>
+        <origin xyz="0.000639 0 0.032486" rpy="0 0 0"/>
+        <mass value="0.656091"/>
+        <inertia ixx="0.0005734" ixy="-2.047e-16" ixz="-3.388729e-6"
+                iyy="0.0006868" iyz="2.988e-16" izz="0.0005789"/>
+      </inertial>
+    </link>
+    <!-- ================= Joint 5 ================= -->
+    <joint name="joint05" type="revolute">
+      <parent link="link05" />
+      <child link="link06" />
+      <origin xyz="0 0 -0.05975" rpy="0 0 0"/>
+      <limit lower="${joint05_lower_limit}" upper="${joint05_upper_limit}" effort="${joint05_effort_limit}" velocity="${joint05_velocity_limit}"/>
+      <axis xyz="1 0 0"/>
+      <dynamics damping="1.0e-6" friction="0.8"/>
+    </joint>
+    <link name="link06">
+      <visual>
+        <origin rpy="3.14159 0 0" xyz="0 0 -0.260"/>
+        <geometry>
+          <mesh filename="package://myrobot_description/meshes/visual/com06.stl" scale="0.001 0.001 0.001"/>
+        </geometry>
+        <material name="${arm_color}"/>
+      </visual>
+      <collision>
+        <origin rpy="3.14159 0 0" xyz="0 0 -0.260"/>
+        <geometry>
+          <mesh filename="package://myrobot_description/meshes/collision/com06.stl" scale="0.001 0.001 0.001"/>
+        </geometry>
+      </collision>
+      <inertial>
+        <origin xyz="-0.00029 0 -0.098217" rpy="0 0 0"/>
+        <mass value="1.560054"/>
+        <inertia ixx="0.01134" ixy="1.01e-15" ixz="3.6208465e-5"
+                iyy="0.01358" iyz="1.59e-15" izz="0.003057"/>
+      </inertial>
+    </link>
+    <!-- ================= Joint 6 ================= -->
+    <joint name="joint06" type="revolute">
+      <parent link="link06" />
+      <child link="link07" />
+      <origin xyz="0 0 -0.260" rpy="0 0 0"/>
+      <limit lower="${joint06_lower_limit}" upper="${joint06_upper_limit}" effort="${joint06_effort_limit}" velocity="${joint06_velocity_limit}"/>
+      <axis xyz="1 0 0"/>
+      <dynamics damping="1.0e-6" friction="0.8"/>
+    </joint>
+    <link name="link07">
+      <visual>
+        <origin rpy="3.14159 0 0" xyz="0 0 -0.2425"/>
+        <geometry>
+          <mesh filename="package://myrobot_description/meshes/visual/com07.stl" scale="0.001 0.001 0.001"/>
+        </geometry>
+        <material name="${arm_color}"/>
+      </visual>
+      <collision>
+        <origin rpy="3.14159 0 0" xyz="0 0 -0.2425"/>
+        <geometry>
+          <mesh filename="package://myrobot_description/meshes/collision/com07.stl" scale="0.001 0.001 0.001"/>
+        </geometry>
+      </collision>
+      <inertial>
+        <origin xyz="-0.000201 -0.00165 -0.051976" rpy="0 0 0"/>
+        <mass value="2.08243"/>
+        <inertia ixx="0.0176" ixy="7.18425e-7" ixz="-2.1360601e-5"
+                iyy="0.0196" iyz="0.0002948" izz="0.00427"/>
+      </inertial>
+    </link>
+    <!-- ================= Joint 7 ================= -->
+    <joint name="joint07" type="revolute">
+      <parent link="link07" />
+      <child link="link08" />
+      <origin xyz="0 0 -0.3099" rpy="0 0 0"/>
+      <limit lower="${joint07_lower_limit}" upper="${joint07_upper_limit}" effort="${joint07_effort_limit}" velocity="${joint07_velocity_limit}"/>
       <axis xyz="0 0 1"/>
       <dynamics damping="1.0e-6" friction="0.8"/>
     </joint>
-    <link name="link6">
-      <visual>
-        <origin rpy="3.14159 0 0" xyz="0 0 0"/>
-        <geometry>
-          <mesh filename="package://myrobot_description/meshes/visual/com6.stl" scale="0.001 0.001 0.001"/>
-        </geometry>
-        <material name="${arm_color}"/>
-      </visual>
-      <collision>
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
File: urdf/myrobot_hand.xacro (robot description, xacro)
@@ -8,9 +8,9 @@
             hand_color
             ">
-    <link name="link10">
+    <link name="hand_link">
       <visual>
         <origin rpy="3.14159 0 1.5708" xyz="0.0 0.0 0.0"/>
         <geometry>
-          <mesh filename="package://myrobot_description/meshes/visual/com10C.stl" scale="0.001 0.001 0.001"/>
+          <mesh filename="package://myrobot_description/meshes/visual/HandMount.stl" scale="0.001 0.001 0.001"/>
         </geometry>
         <material name="${hand_color}"/>
@@ -19,15 +19,16 @@
         <origin rpy="3.14159 0 1.5708" xyz="0.0 0.0 0.0"/>
         <geometry>
-          <mesh filename="package://myrobot_description/meshes/collision/com10C.stl" scale="0.001 0.001 0.001"/>
+          <mesh filename="package://myrobot_description/meshes/collision/HandMount.stl" scale="0.001 0.001 0.001"/>
         </geometry>
       </collision>
       <inertial>
-        <origin rpy="1.5708 0 0" xyz="-0.118e-03 -20.65e-03 1.006e-03"/>
-        <inertia ixx="32600.928e-09" ixy="-69.84e-09" ixz="-254.224e-09" iyy="41969.484e-09" iyz="-409.16e-09" izz="43040.018e-09"/>
-        <mass value="121.0e-03"/>
+        <origin xyz="0.00036 -0.00003 0.018185" rpy="0 0 0"/>
+        <mass value="0.164186"/>
+        <inertia ixx="5.5155958e-5" ixy="-6.0872e-8" ixz="-1.9987e-7"
+                iyy="7.2198073e-5" iyz="3.7257e-8" izz="7.8575254e-5"/>
       </inertial>
     </link>
-    <joint name="hand_joint" type="revolute">
-      <parent link="link10" />
+    <joint name="joint_grip" type="revolute">
+      <parent link="hand_link" />
       <child link="handA_link" />
       <origin xyz="0.0 -0.012 -0.02575" rpy="0 0 0"/>
@@ -44,5 +45,5 @@
         <origin rpy="3.14159 0 -1.5708" xyz="0.0 0.0 0.0"/>
         <geometry>
-          <mesh filename="package://myrobot_description/meshes/visual/com10A.stl" scale="0.001 0.001 0.001"/>
+          <mesh filename="package://myrobot_description/meshes/visual/HandFingureA.stl" scale="0.001 0.001 0.001"/>
         </geometry>
         <material name="${hand_color}"/>
@@ -51,15 +52,16 @@
         <origin rpy="3.14159 0 -1.5708" xyz="0.0 0.0 0.0"/>
         <geometry>
-          <mesh filename="package://myrobot_description/meshes/collision/com10A.stl" scale="0.001 0.001 0.001"/>
+          <mesh filename="package://myrobot_description/meshes/collision/HandFingureA.stl" scale="0.001 0.001 0.001"/>
         </geometry>
       </collision>
       <inertial>
-        <origin rpy="0 0 0" xyz="2.649e-03 -26.849e-03 3.757e-03"/>
-        <inertia ixx="10192.75e-09" ixy="-197.895e-09" ixz="98.609e-09" iyy="5023.728e-09" iyz="-554.407e-09" izz="6322.202e-09"/>
-        <mass value="15.8e-03"/>
+        <origin xyz="-0.001325 -3.967e-10 0.022033" rpy="0 0 0"/>
+        <mass value="0.020568"/>
+        <inertia ixx="1.0584193e-5" ixy="-1.041e-14" ixz="5.62926e-7"
+                iyy="4.874099e-6" iyz="0" izz="6.957021e-6"/>
       </inertial>
     </link>
-    <joint name="hand_mimic_joint" type="revolute">
-      <parent link="link10" />
+    <joint name="joint_grip_mimic" type="revolute">
+      <parent link="hand_link" />
       <child link="handB_link" />
       <origin xyz="0.0 0.012 -0.02575" rpy="0 0 0"/>
@@ -70,5 +72,5 @@
         velocity="${hand_joints_velocity_limit}"/>
       <axis xyz="-1 0 0"/>
-      <mimic joint="hand_joint" multiplier="1" offset="0"/>
+      <mimic joint="joint_grip" multiplier="1" offset="0"/>
       <dynamics damping="1.0e-6" friction="0.8"/>
     </joint>
@@ -77,5 +79,5 @@
         <origin rpy="3.14159 0 -1.5708" xyz="0.0 0.0 0.0"/>
         <geometry>
-          <mesh filename="package://myrobot_description/meshes/visual/com10B.stl" scale="0.001 0.001 0.001"/>
+          <mesh filename="package://myrobot_description/meshes/visual/HandFingureB.stl" scale="0.001 0.001 0.001"/>
         </geometry>
         <material name="${hand_color}"/>
@@ -84,14 +86,15 @@
         <origin rpy="3.14159 0 -1.5708" xyz="0.0 0.0 0.0"/>
         <geometry>
-          <mesh filename="package://myrobot_description/meshes/collision/com10B.stl" scale="0.001 0.001 0.001"/>
+          <mesh filename="package://myrobot_description/meshes/collision/HandFingureB.stl" scale="0.001 0.001 0.001"/>
         </geometry>
       </collision>
       <inertial>
-        <origin rpy="0 0 0" xyz="-2.707e-03 -30.901e-03 2.845e-03"/>
-        <inertia ixx="7483.7e-09" ixy="361.283e-09" ixz="-63.385e-09" iyy="4088.581e-09" iyz="-228.226e-09" izz="4372.991e-09"/>
-        <mass value="13.9e-03"/>
+        <origin xyz="0.001385 -0.000244 0.021686" rpy="0 0 0"/>
+        <mass value="0.02096"/>
+        <inertia ixx="1.0837944e-5" ixy="-7.082e-9" ixz="-5.33588e-7"
+                iyy="5.007456e-6" iyz="-1.10875e-7" izz="7.078359e-6"/>
       </inertial>
     </link>
-    <gazebo reference="link10">
+    <gazebo reference="hand_link">
       <material>Gazebo/Red</material>
     </gazebo>
