Commit message: v1 : arm failed to move due to excessive weight

File: urdf/myrobot.urdf.xacro (robot description, xacro)
@@ -44,5 +44,5 @@
       <xacro:default_transmission joint_name="joint08" interface="${right_arm_interface}"/>
       <xacro:default_transmission joint_name="joint09" interface="${right_arm_interface}"/>
-      <xacro:default_transmission joint_name="joint_grip" interface="position"/>
+      <xacro:default_transmission joint_name="hand_joint" interface="position"/>
     </xacro:if>
   </xacro:if>
@@ -51,8 +51,8 @@
 	<!-- connect base and world via three axes expressing mobile platform -->
 	<link name="base_link"/>
-	<joint name="base_fixed_joint" type="fixed">
+	<joint name="joint_base-to-world" type="fixed">
     <parent link="world"/>
     <child link="base_link"/>
-    <origin xyz="0 0 1.5" rpy="0 0 0"/>
+    <origin xyz="0 0 0" rpy="0 0 0"/>
   </joint>
   <xacro:myrobot
@@ -75,12 +75,12 @@
     joint09_lower_limit="${radians(-90)}"
     joint09_upper_limit="${radians(90)}"
-    joint01_effort_limit  ="${XH430_V350_EFFORT_LIMIT}"
-    joint01_velocity_limit="${XH430_V350_VELOCITY_LIMIT}"
-    joint02_effort_limit  ="${XH430_V350_EFFORT_LIMIT}"
-    joint02_velocity_limit="${XH430_V350_VELOCITY_LIMIT}"
-    joint03_effort_limit  ="${XH430_V350_EFFORT_LIMIT}"
-    joint03_velocity_limit="${XH430_V350_VELOCITY_LIMIT}"
-    joint04_effort_limit  ="${XH430_V350_EFFORT_LIMIT}"
-    joint04_velocity_limit="${XH430_V350_VELOCITY_LIMIT}"
+    joint01_effort_limit  ="${RMD_X4_P36_36_E_EFFORT_LIMIT}"
+    joint01_velocity_limit="${RMD_X4_P36_36_E_VELOCITY_LIMIT}"
+    joint02_effort_limit  ="${RMD_X4_P36_36_E_EFFORT_LIMIT}"
+    joint02_velocity_limit="${RMD_X4_P36_36_E_VELOCITY_LIMIT}"
+    joint03_effort_limit  ="${RMD_X4_P36_36_E_EFFORT_LIMIT}"
+    joint03_velocity_limit="${RMD_X4_P36_36_E_VELOCITY_LIMIT}"
+    joint04_effort_limit  ="${RMD_X4_P36_36_E_EFFORT_LIMIT}"
+    joint04_velocity_limit="${RMD_X4_P36_36_E_VELOCITY_LIMIT}"
     joint05_effort_limit  ="${XH430_V350_EFFORT_LIMIT}"
     joint05_velocity_limit="${XH430_V350_VELOCITY_LIMIT}"
@@ -98,5 +98,5 @@
     hand_joints_lower_limit="${radians(-90)}"
     hand_joints_upper_limit="${radians(0)}"
-    hand_joints_effort_limit ="${XH430_V350_EFFORT_LIMIT}"
+    hand_joints_effort_limit  ="${XH430_V350_EFFORT_LIMIT}"
     hand_joints_velocity_limit="${XH430_V350_VELOCITY_LIMIT}"
     hand_color="red">

File: urdf/myrobot.xacro (robot description, xacro)
@@ -26,5 +26,5 @@
       <parent link="base_link" />
       <child link="link01" />
-      <origin xyz="0 0 0" rpy="0 0 0"/>
+      <origin xyz="0 0 1.5" rpy="0 0 1.5708"/>
     </joint>
     <link name="link01">
@@ -43,7 +43,13 @@
       </collision>
       <inertial>
-        <origin rpy="0 0 0" xyz="0 0 0"/>
-        <inertia ixx="1e-4" ixy="0" ixz="0" iyy="1e-4" iyz="0" izz="1e-4"/>
-        <mass value="0.25"/>
+        <origin xyz="0.0 0.0 0.033626" rpy="0 0 0"/>
+        <mass value="0.955929"/>
+        <inertia
+          ixx="0.0009194"
+          ixy="0.0"
+          ixz="-7.677e-12"
+          iyy="0.0009194"
+          iyz="2.373e-13"
+          izz="0.001105"/>
       </inertial>
     </link>
@@ -72,7 +78,13 @@
       </collision>
       <inertial>
-        <origin rpy="0 0 0" xyz="0 0 0"/>
-        <inertia ixx="1e-4" ixy="0" ixz="0" iyy="1e-4" iyz="0" izz="1e-4"/>
-        <mass value="0.2"/>
+        <origin xyz="-6.648e-13 0.000189 0.050235" rpy="0 0 0"/>
+        <mass value="0.972294"/>
+        <inertia
+          ixx="0.001458"
+          ixy="-8.837e-15"
+          ixz="0.0"
+          iyy="0.001420"
+          iyz="-2.259128e-6"
+          izz="0.0008793"/>
       </inertial>
     </link>
@@ -81,5 +93,5 @@
       <parent link="link02" />
       <child link="link03" />
-      <origin xyz="0 0 -0.0715" rpy="0 0 0"/>
+      <origin xyz="0 0 -0.080" rpy="0 0 0"/>
       <limit lower="${joint02_lower_limit}" upper="${joint02_upper_limit}" effort="${joint02_effort_limit}" velocity="${joint02_velocity_limit}"/>
       <axis xyz="0 1 0"/>
@@ -101,7 +113,13 @@
       </collision>
       <inertial>
-        <origin rpy="0 0 0" xyz="0 0 0"/>
-        <inertia ixx="1e-4" ixy="0" ixz="0" iyy="1e-4" iyz="0" izz="1e-4"/>
-        <mass value="0.2"/>
+        <origin xyz="2.151e-12 -0.000093 0.13806" rpy="0 0 0"/>
+        <mass value="2.085173"/>
+        <inertia
+          ixx="0.007892"
+          ixy="-1.581e-15"
+          ixz="1.0e-12"
+          iyy="0.007836"
+          iyz="-2.6867331e-5"
+          izz="0.002416"/>
       </inertial>
     </link>
@@ -110,5 +128,5 @@
       <parent link="link03"/>
       <child link="link04"/>
-      <origin xyz="0 0 -0.0715" rpy="0 0 0"/>
+      <origin xyz="0 0 -0.2265" rpy="0 0 0"/>
       <limit lower="${joint03_lower_limit}" upper="${joint03_upper_limit}" effort="${joint03_effort_limit}" velocity="${joint03_velocity_limit}"/>
       <axis xyz="0 0 1"/>
@@ -130,7 +148,13 @@
       </collision>
       <inertial>
-        <origin rpy="0 0 0" xyz="0 0 0"/>
-        <inertia ixx="1e-4" ixy="0" ixz="0" iyy="1e-4" iyz="0" izz="1e-4"/>
-        <mass value="0.2"/>
+        <origin xyz="1.397e-12 -0.000102 0.082913" rpy="0 0 0"/>
+        <mass value="1.805227"/>
+        <inertia
+          ixx="0.005333"
+          ixy="-1.062e-14"
+          ixz="0.0"
+          iyy="0.005295"
+          iyz="9.107951e-6"
+          izz="0.001938"/>
       </inertial>
     </link>
@@ -159,7 +183,13 @@
       </collision>
       <inertial>
-        <origin rpy="0 0 0" xyz="0 0 0"/>
-        <inertia ixx="1e-4" ixy="0" ixz="0" iyy="1e-4" iyz="0" izz="1e-4"/>
-        <mass value="0.2"/>
+        <origin xyz="-1.552e-8 -0.000458 0.11458" rpy="0 0 0"/>
+        <mass value="1.496725"/>
+        <inertia
+          ixx="0.004471"
+          ixy="-1.141e-9"
+          ixz="1.313e-9"
+          iyy="0.004431"
+          iyz="8.1422738e-5"
+          izz="0.001787"/>
       </inertial>
     </link>
@@ -188,7 +218,13 @@
       </collision>
       <inertial>
-        <origin rpy="0 0 0" xyz="0 0 0"/>
-        <inertia ixx="1e-4" ixy="0" ixz="0" iyy="1e-4" iyz="0" izz="1e-4"/>
-        <mass value="0.15"/>
+        <origin xyz="1.95e-12 -0.000008 0.040157" rpy="0 0 0"/>
+        <mass value="0.646831"/>
+        <inertia
+          ixx="0.0006439"
+          ixy="-2.594e-16"
+          ixz="7.915e-15"
+          iyy="0.0006524"
+          iyz="2.46697e-7"
+          izz="0.00063"/>
       </inertial>
     </link>
@@ -217,7 +253,13 @@
       </collision>
       <inertial>
-        <origin rpy="0 0 0" xyz="0 0 0"/>
-        <inertia ixx="1e-4" ixy="0" ixz="0" iyy="1e-4" iyz="0" izz="1e-4"/>
-        <mass value="0.1"/>
+        <origin xyz="0.000019 0.000721 0.073717" rpy="0 0 0"/>
+        <mass value="1.221822"/>
+        <inertia
+          ixx="0.001959"
+          ixy="-1.135e-9"
+          ixz="-7.53e-10"
+          iyy="0.001954"
+          iyz="-3.7865055e-5"
+          izz="0.001725"/>
       </inertial>
     </link>
@@ -246,7 +288,13 @@
       </collision>
       <inertial>
-        <origin rpy="0 0 0" xyz="0 0 0"/>
-        <inertia ixx="1e-4" ixy="0" ixz="0" iyy="1e-4" iyz="0" izz="1e-4"/>
-        <mass value="0.1"/>
+        <origin xyz="1.95e-12 -0.000008 0.040157" rpy="0 0 0"/>
+        <mass value="0.646831"/>
+        <inertia
+          ixx="0.0006439"
+          ixy="-2.594e-16"
+          ixz="7.915e-15"
+          iyy="0.0006524"
+          iyz="2.46697e-7"
+          izz="0.00063"/>
       </inertial>
     </link>
@@ -275,7 +323,13 @@
       </collision>
       <inertial>
-        <origin rpy="0 0 0" xyz="0 0 0"/>
-        <inertia ixx="1e-4" ixy="0" ixz="0" iyy="1e-4" iyz="0" izz="1e-4"/>
-        <mass value="0.1"/>
+        <origin xyz="-0.000019 -0.000721 0.073717" rpy="0 0 0"/>
+        <mass value="1.221822"/>
+        <inertia
+          ixx="0.001959"
+          ixy="-1.135e-9"
+          ixz="7.53e-10"
+          iyy="0.001954"
+          iyz="3.7865055e-5"
+          izz="0.001725"/>
       </inertial>
     </link>
@@ -283,6 +337,6 @@
     <joint name="joint09" type="revolute">
       <parent link="link09" />
-      <child link="hand_link" />
-      <origin xyz="0 0 -0.14050" rpy="0 0 0"/>
+      <child link="HandMount_link" />
+      <origin xyz="0 0 -0.1355" rpy="0 0 0"/>
       <limit lower="${joint09_lower_limit}" upper="${joint09_upper_limit}" effort="${joint09_effort_limit}" velocity="${joint09_velocity_limit}"/>
       <axis xyz="0 0 1"/>

File: urdf/myrobot_hand.xacro (robot description, xacro)
@@ -8,5 +8,5 @@
             hand_color
             ">
-    <link name="hand_link">
+    <link name="HandMount_link">
       <visual>
         <origin rpy="3.14159 0 1.5708" xyz="0.0 0.0 0.0"/>
@@ -23,12 +23,19 @@
       </collision>
       <inertial>
-        <origin rpy="1.5708 0 0" xyz="-0.118e-03 -20.65e-03 1.006e-03"/>
-        <inertia ixx="32600.928e-09" ixy="-69.84e-09" ixz="-254.224e-09" iyy="41969.484e-09" iyz="-409.16e-09" izz="43040.018e-09"/>
-        <mass value="121.0e-03"/>
+        <origin xyz="0.000264 -0.000049 0.023304" rpy="0 0 0"/>
+        <mass value="0.205541"/>
+        <inertia
+          ixx="0.000095997183"
+          ixy="-1.231e-7"
+          ixz="1.41185e-7"
+          iyy="0.0001288"
+          iyz="2.4556e-8"
+          izz="0.0001199"/>
       </inertial>
     </link>
+    <!-- ================= Joint hand mount to HandFingerA_link ================= -->
     <joint name="hand_joint" type="revolute">
-      <parent link="hand_link" />
-      <child link="handA_link" />
+      <parent link="HandMount_link" />
+      <child link="HandFingerA_link" />
       <origin xyz="0.0 -0.012 -0.02575" rpy="0 0 0"/>
       <limit
@@ -40,5 +47,5 @@
       <dynamics damping="1.0e-6" friction="0.8"/>
     </joint>
-    <link name="handA_link">
+    <link name="HandFingerA_link">
       <visual>
         <origin rpy="3.14159 0 -1.5708" xyz="0.0 0.0 0.0"/>
@@ -55,12 +62,19 @@
       </collision>
       <inertial>
-        <origin rpy="0 0 0" xyz="2.649e-03 -26.849e-03 3.757e-03"/>
-        <inertia ixx="10192.75e-09" ixy="-197.895e-09" ixz="98.609e-09" iyy="5023.728e-09" iyz="-554.407e-09" izz="6322.202e-09"/>
-        <mass value="15.8e-03"/>
+        <origin xyz="-0.001325 -3.967e-10 0.022033" rpy="0 0 0"/>
+        <mass value="0.020568"/>
+        <inertia
+          ixx="0.000010584193"
+          ixy="-1.041e-14"
+          ixz="5.62926e-7"
+          iyy="0.000004874099"
+          iyz="0.0"
+          izz="0.000006957021"/>
       </inertial>
     </link>
-    <joint name="hand_joint_mimic" type="revolute">
-      <parent link="hand_link" />
-      <child link="handB_link" />
+    <!-- ================= Joint hand finger B to hand fingerA ================= -->
+    <joint name="hand_mimic_joint" type="revolute">
+      <parent link="HandMount_link" />
+      <child link="HandFingerB_link" />
       <origin xyz="0.0 0.012 -0.02575" rpy="0 0 0"/>
       <limit
@@ -73,5 +87,5 @@
       <dynamics damping="1.0e-6" friction="0.8"/>
     </joint>
-    <link name="handB_link">
+    <link name="HandFingerB_link">
       <visual>
         <origin rpy="3.14159 0 -1.5708" xyz="0.0 0.0 0.0"/>
@@ -88,16 +102,22 @@
       </collision>
       <inertial>
-        <origin rpy="0 0 0" xyz="-2.707e-03 -30.901e-03 2.845e-03"/>
-        <inertia ixx="7483.7e-09" ixy="361.283e-09" ixz="-63.385e-09" iyy="4088.581e-09" iyz="-228.226e-09" izz="4372.991e-09"/>
-        <mass value="13.9e-03"/>
+        <origin xyz="0.001385 -0.000244 0.021686" rpy="0 0 0"/>
+        <mass value="0.02096"/>
+        <inertia
+          ixx="0.000010837944"
+          ixy="-7.082e-9"
+          ixz="-5.33588e-7"
+          iyy="0.000005007456"
+          iyz="-1.10875e-7"
+          izz="0.000007078359"/>
       </inertial>
     </link>
-    <gazebo reference="hand_link">
+    <gazebo reference="HandMount_link">
       <material>Gazebo/Red</material>
     </gazebo>
-    <gazebo reference="handA_link">
+    <gazebo reference="HandFingerA_link">
       <material>Gazebo/Red</material>
     </gazebo>
-    <gazebo reference="handB_link">
+    <gazebo reference="HandFingerB_link">
       <material>Gazebo/Red</material>
     </gazebo>
